File: KIcad/Smart Ventilator PCB.kicad_pcb (KiCad board)
At the start: 2 copper layers, 204 x 179 mm, 54 parts, among them J1 Conn_01x07_Female, J2 Screw_Terminal_01x12, J3 Screw_Terminal_01x03, J4 Conn_01x04_Female, J5 Conn_01x06_Female, K1 DIPxx-1Axx-11x, K2 DIPxx-1Axx-11x, Q1 TIP41, Q2 TIP41, Q3 TIP41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

Commit message: PCB Added
Parts:
- removed REF** (x6): MountingHole_2.1mm, MountingHole:MountingHole_2.1mm
- added C4: 470uF, Capacitor_SMD:C_Elec_3x5.4, F.Cu at (211.3, 131.1)
- added C5: 2200uF, Capacitor_SMD:C_Elec_5x5.4, F.Cu at (232.7, 96.1)
- added C6: 470uF, Capacitor_SMD:C_Elec_3x5.4, F.Cu at (248.8, 123.1)
- added C7: 470uF, Capacitor_SMD:C_Elec_3x5.4, F.Cu at (248.5, 96.1)
- added C8: 470uF, Capacitor_SMD:C_Elec_3x5.4, F.Cu at (248.8, 105.3)
- added C9: 470uF, Capacitor_SMD:C_Elec_3x5.4, F.Cu at (248.8, 112.9)
- added D5: ABS4, Diode_SMD:Diode_Bridge_Diotec_ABS, F.Cu at (220.4, 108.9)
- added D6: LED, LED_SMD:LED_0603_1608Metric_Pad1.05x0.95mm_HandSolder, F.Cu at (210.5, 107.2)
- added D7: 1N4004, Diode_THT:D_DO-41_SOD81_P10.16mm_Horizontal, F.Cu at (241.1, 106.7)
- added D8: 1N4004, Diode_THT:D_DO-41_SOD81_P10.16mm_Horizontal, F.Cu at (203.7, 102.7)
- added IC1: L7805, footprint:78XXL, F.Cu at (199.0, 117.7)
- added IC2: L7805, footprint:78XXL, F.Cu at (222.2, 137.5)
- added J6: Screw_Terminal_01x05, TerminalBlock_4Ucon:TerminalBlock_4Ucon_1x05_P3.50mm_Horizontal, F.Cu at (227.6, 86.5)
- added J7: Screw_Terminal_01x05, TerminalBlock_4Ucon:TerminalBlock_4Ucon_1x05_P3.50mm_Horizontal, F.Cu at (231.5, 152.8)
- added J8: Conn_01x01_Female, Connector_PinHeader_1.00mm:PinHeader_1x01_P1.00mm_Vertical, F.Cu at (208.8, 152.9)
- added R4: 1.6k, Resistor_THT:R_Axial_DIN0207_L6.3mm_D2.5mm_P10.16mm_Horizontal, F.Cu at (198.1, 92.4)
- added R5: 1k, Resistor_THT:R_Axial_DIN0207_L6.3mm_D2.5mm_P10.16mm_Horizontal, F.Cu at (232.7, 113.4)
- added T1: Transformer_1P_1S, Transformer_SMD:Pulse_PA2006NL, F.Cu at (220.1, 96.6)
- added U10: OKI-78SR-3.3_1.5-W36-C, Converter_DCDC:Converter_DCDC_Murata_OKI-78SR_Vertical, F.Cu at (229.8, 122.0)
- added U11: R-7812-0.5, Converter_DCDC:Converter_DCDC_RECOM_R-78E-0.5_THT, F.Cu at (214.1, 123.6)
- added U9: LD1086DT18TR, Package_TO_SOT_SMD:TO-252-2, F.Cu at (246.7, 135.4)
- 1k1, 1k2, 1k3, 1k4, 1k5, 1k6, 1k7, 1k8, R1, R2, R3: footprint Resistor_SMD:R_0201_0603Metric -> Resistor_THT:R_Axial_DIN0207_L6.3mm_D2.5mm_P10.16mm_Horizontal
- SW1, SW2: footprint Button_Switch_SMD:SW_Push_1P1T-MP_NO_Horizontal_Alps_SKRTLAE010 -> Button_Switch_SMD:SW_Push_1P1T_NO_6x6mm_H9.5mm
- U5, U6: value MPX4250 -> MPX4250AP; footprint Sensor:Aosong_DHT11_5.5x12.0_P2.54mm -> footprint:MPX4250AP
- Y1: moved to B.Cu
- moved Q1 107.7 mm to (93.3, 140.9)
- moved U5 64.3 mm to (81.5, 94.0), turned to -90 degrees
- moved K2 64.0 mm to (53.2, 43.4)
- moved BZ1 61.6 mm to (60.4, 118.1)
- moved U3 56.2 mm to (74.9, 138.1), turned to 180 degrees
- moved RV2 39.5 mm to (46.7, 127.1)
- moved U8 30.7 mm to (182.9, 62.6)
- moved RV1 30.0 mm to (37.7, 126.8)
- moved U4 29.2 mm to (62.5, 104.8), turned to 180 degrees
- moved U6 29.0 mm to (81.5, 54.0), turned to -90 degrees
- moved 1k5 28.7 mm to (39.9, 83.0)
- moved D3 26.1 mm to (31.5, 48.7)
- moved D1 25.9 mm to (37.0, 48.9)
- moved 1k8 25.5 mm to (174.4, 70.3), turned to 90 degrees
- moved D2 23.9 mm to (31.6, 52.7)
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Routing:
- net +5V: track 0.00 -> 339.3 mm, vias 0 -> 12
- net /Power Supply/Battery -: track 0.00 -> 200.9 mm, vias 0 -> 8
- net Net-(C4-Pad1): track 0.00 -> 151.7 mm, vias 0 -> 1
- net Net-(1k1-Pad2): track 0.00 -> 143.0 mm
- net Net-(C6-Pad1): track 0.00 -> 141.1 mm, vias 0 -> 2
- net GND: track 0.00 -> 132.9 mm, vias 0 -> 17
- net /stepper 14: track 0.00 -> 125.5 mm, vias 0 -> 2
- net /stepper 3: track 0.00 -> 121.0 mm, vias 0 -> 3
- net /stepper 4: track 0.00 -> 109.8 mm, vias 0 -> 5
- net Net-(U1-Pad40): track 0.00 -> 109.4 mm
- net /SDA: track 0.00 -> 109.0 mm, vias 0 -> 4
- net Net-(22pF2-Pad1): track 0.00 -> 107.9 mm, vias 0 -> 4
- net Net-(U1-Pad41): track 0.00 -> 105.8 mm
- net /stepper 11: track 0.00 -> 104.6 mm, vias 0 -> 4
- net /SCL: track 0.00 -> 104.2 mm, vias 0 -> 4
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- added copper zone on B.Cu, net GND
- added copper zone on F.Cu, net GND
Other:
- board size 204 x 179 mm -> 240 x 179.5 mm
